File: mbes_inputs.kicad_sch (KiCad schematic)
At the start: 7 parts

Commit message: First release of all-in-one solution
Parts:
- added KeyLocker1: Conn_01x08, Connector_PinHeader_2.54mm:PinHeader_1x08_P2.54mm_Vertical, symbol Connector_Generic:Conn_01x08
- added R1: 500, Resistor_THT:R_Axial_DIN0309_L9.0mm_D3.2mm_P12.70mm_Horizontal, symbol Device:R
- gave numbers to parts that had none: 7
Connections:
- net GND: now also rightCtrls_conn1.1 (Pin_1); no longer rightCtrls_conn1.4 (Pin_4)
- net i_startButton: now also rightCtrls_conn1.4 (Pin_4); no longer rightCtrls_conn1.1 (Pin_1)
- net i_engineOFF renamed c_engineOFF
- new net: KeyLocker1.1 (Pin_1), KeyLocker1.3 (Pin_3), R1.2
- new net +5V: KeyLocker1.8 (Pin_8)
- new net i_Vx1: KeyLocker1.2 (Pin_2)
- new net i_Vx2: KeyLocker1.4 (Pin_4)
- new net tempPower: KeyLocker1.7 (Pin_7), R1.1
- no-connect marks 0 -> 2
