File: PCB/motorbike_electrical_system.kicad_sch (KiCad schematic)
At the start: 10 parts, among them U1 L7805, U2 L7805, U3 L7805, U4 ATmega16L-8P

Commit message: External cockpit power-connector added and wrong transistor type fixed
Connections:
- net i_powerOFF: now also U4.9 (~{RESET}); no longer U4.26 (PC4)
- net tempPower: now also U4.30 (AVCC)
- no-connect marks 7 -> 6
Changed lines of the file:
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@@
   (junction (at 37.211 185.42) (diameter 0) (color 0 0 0 0)
   )
+  (junction (at 127.4064 44.704) (diameter 0) (color 0 0 0 0)
+  )
   (junction (at 108.3564 176.53) (diameter 0) (color 0 0 0 0)
   )
@@
   (junction (at 62.484 169.672) (diameter 0) (color 0 0 0 0)
   )
-  (no_connect (at 112.141 59.182))
-  (no_connect (at 112.141 69.342))
-  (no_connect (at 112.141 64.262))
-  (no_connect (at 129.921 46.482))
-  (no_connect (at 142.621 66.802))
-  (no_connect (at 112.141 54.102))
-  (no_connect (at 142.621 64.262))
+  (no_connect (at 112.1664 59.182))
+  (no_connect (at 112.1664 69.342))
+  (no_connect (at 142.6464 109.982))
+  (no_connect (at 112.1664 64.262))
+  (no_connect (at 142.6464 66.802))
+  (no_connect (at 142.6464 64.262))
   (wire (pts (xy 173.482 146.4564) (xy 151.638 146.4564))
     (stroke (width 0) (type default) (color 0 0 0 0))
   )
-  (wire (pts (xy 142.6464 109.982) (xy 149.1488 109.982))
-    (stroke (width 0) (type default) (color 0 0 0 0))
-  )
   (wire (pts (xy 191.4144 63.1952) (xy 191.4144 56.7944))
     (stroke (width 0) (type default) (color 0 0 0 0))
@@
     (stroke (width 0) (type default) (color 0 0 0 0))
   )
-  (wire (pts (xy 127.4064 39.37) (xy 127.4064 46.482))
+  (wire (pts (xy 127.4064 39.37) (xy 127.4064 44.704))
     (stroke (width 0) (type default) (color 0 0 0 0))
   )
@@
     (stroke (width 0) (type default) (color 0 0 0 0))
   )
-  (wire (pts (xy 149.1488 109.982) (xy 149.1488 111.6584))
-    (stroke (width 0) (type default) (color 0 0 0 0))
-  )
   (wire (pts (xy 174.9044 147.8788) (xy 149.9616 147.8788))
     (stroke (width 0) (type default) (color 0 0 0 0))
@@
     (stroke (width 0) (type default) (color 0 0 0 0))
   )
+  (wire (pts (xy 127.4064 44.704) (xy 127.4064 46.482))
+    (stroke (width 0) (type default) (color 0 0 0 0))
+  )
   (wire (pts (xy 149.1488 102.362) (xy 149.1488 101.5492))
     (stroke (width 0) (type default) (color 0 0 0 0))
@@
     (stroke (width 0) (type default) (color 0 0 0 0))
   )
+  (wire (pts (xy 129.9464 44.704) (xy 127.4064 44.704))
+    (stroke (width 0) (type default) (color 0 0 0 0))
+  )
   (wire (pts (xy 142.6464 125.222) (xy 154.5844 125.222))
     (stroke (width 0) (type default) (color 0 0 0 0))
@@
     (stroke (width 0) (type default) (color 0 0 0 0))
   )
+  (wire (pts (xy 99.822 54.102) (xy 112.1664 54.102))
+    (stroke (width 0) (type default) (color 0 0 0 0))
+  )
   (wire (pts (xy 197.9168 47.7012) (xy 204.7748 47.7012))
     (stroke (width 0) (type default) (color 0 0 0 0))
@@
     (stroke (width 0) (type default) (color 0 0 0 0))
   )
-  (wire (pts (xy 149.1488 111.6584) (xy 157.988 111.6584))
-    (stroke (width 0) (type default) (color 0 0 0 0))
-  )
   (wire (pts (xy 179.9844 129.3368) (xy 171.0944 129.3368))
     (stroke (width 0) (type default) (color 0 0 0 0))
@@
   )
   (wire (pts (xy 155.956 122.682) (xy 142.6464 122.682))
+    (stroke (width 0) (type default) (color 0 0 0 0))
+  )
+  (wire (pts (xy 129.9464 46.482) (xy 129.9464 44.704))
     (stroke (width 0) (type default) (color 0 0 0 0))
   )
@@
     )
   )
-  (global_label "i_powerOFF" (shape input) (at 157.988 111.6584 0) (fields_autoplaced)
-    (effects (font (size 1.27 1.27)) (justify left))
-    (property "Riferimenti inter-foglio" "${INTERSHEET_REFS}" (id 0) (at 170.9844 111.579 0)
-      (effects (font (size 1.27 1.27)) (justify left) hide)
+  (global_label "i_powerOFF" (shape input) (at 99.822 54.102 180) (fields_autoplaced)
+    (effects (font (size 1.27 1.27)) (justify right))
+    (property "Riferimenti inter-foglio" "${INTERSHEET_REFS}" (id 0) (at 86.8256 54.1814 0)
+      (effects (font (size 1.27 1.27)) (justify right) hide)
     )
   )
@@
       (reference "#PWR0108") (unit 1) (value "GND") (footprint "")
     )
+    (path "/44e17612-9f2f-476d-8e41-268bb036a54a/d5040709-02aa-4b57-873b-3227ea381679"
+      (reference "#PWR0109") (unit 1) (value "GND") (footprint "")
+    )
+    (path "/44e17612-9f2f-476d-8e41-268bb036a54a/a0b371de-a4a3-4f8b-a3f2-34b9eb0e50e3"
+      (reference "#PWR0110") (unit 1) (value "+12V") (footprint "")
+    )
     (path "/44e17612-9f2f-476d-8e41-268bb036a54a/ca96e50f-3e2b-4429-a303-34aeefffd5a5"
       (reference "Arrow_p1") (unit 1) (value "Conn_01x03") (footprint "Connector_Wire:SolderWire-1.5sqmm_1x03_P6mm_D1.7mm_OD3mm")
@@
       (reference "Q15") (unit 1) (value "D45VH10") (footprint "Package_TO_SOT_THT:TO-220-3_Vertical")
     )
-    (path "/44e17612-9f2f-476d-8e41-268bb036a54a/0941dfe8-e905-4160-932a-17fff6ee0d8c"
+    (path "/44e17612-9f2f-476d-8e41-268bb036a54a/3afa411e-2443-4a91-8e43-4f2e8144928e"
       (reference "Q16") (unit 1) (value "BC337") (footprint "Package_TO_SOT_THT:TO-92L_Inline_Wide")
     )
@@
       (reference "Q17") (unit 1) (value "BC337") (footprint "Package_TO_SOT_THT:TO-92L_Inline_Wide")
     )
+    (path "/44e17612-9f2f-476d-8e41-268bb036a54a/4ebf1fdd-474b-40f8-ba13-dc71aa6f2221"
+      (reference "Q18") (unit 1) (value "BC327") (footprint "Package_TO_SOT_THT:TO-92L_Inline_Wide")
+    )
+    (path "/44e17612-9f2f-476d-8e41-268bb036a54a/1bd668b1-fa3d-4d0c-92f2-a210f19649fa"
+      (reference "Q19") (unit 1) (value "BC327") (footprint "Package_TO_SOT_THT:TO-92L_Inline_Wide")
+    )
+    (path "/44e17612-9f2f-476d-8e41-268bb036a54a/689c51fd-5eab-4f64-8671-f087ef7fe018"
+      (reference "Q20") (unit 1) (value "BC327") (footprint "Package_TO_SOT_THT:TO-92L_Inline_Wide")
+    )
     (path "/0b22d592-b723-42a2-89dd-bec665c2bd26/b8448d20-86fe-4c18-8be5-bf46157011d9"
       (reference "R1") (unit 1) (value "500") (footprint "Resistor_THT:R_Axial_DIN0309_L9.0mm_D3.2mm_P12.70mm_Horizontal")
@@
       (reference "RA44") (unit 1) (value "100K") (footprint "Resistor_THT:R_Axial_DIN0207_L6.3mm_D2.5mm_P7.62mm_Horizontal")
     )
+    (path "/44e17612-9f2f-476d-8e41-268bb036a54a/d32e5412-d9b7-4bbb-8c22-8d1adfe183d3"
+      (reference "RA45") (unit 1) (value "10K") (footprint "Resistor_THT:R_Axial_DIN0207_L6.3mm_D2.5mm_P7.62mm_Horizontal")
+    )
+    (path "/44e17612-9f2f-476d-8e41-268bb036a54a/03e01814-a676-45c6-8c54-822d432e2a2c"
+      (reference "RA46") (unit 1) (value "3K") (footprint "Resistor_THT:R_Axial_DIN0207_L6.3mm_D2.5mm_P7.62mm_Horizontal")
+    )
+    (path "/44e17612-9f2f-476d-8e41-268bb036a54a/e0f35305-9e12-4295-82b7-0cee6273f340"
+      (reference "RA47") (unit 1) (value "3K") (footprint "Resistor_THT:R_Axial_DIN0207_L6.3mm_D2.5mm_P7.62mm_Horizontal")
+    )
     (path "/dfeffa1f-9119-4780-8aed-ab76c9242c17"
       (reference "RV1") (unit 1) (value "10K") (footprint "Potentiometer_THT:Potentiometer_Bourns_3296W_Vertical")
@@
       (reference "addLights1") (unit 1) (value "Conn_01x02") (footprint "Connector_PinSocket_2.54mm:PinSocket_1x02_P2.54mm_Vertical")
     )
+    (path "/44e17612-9f2f-476d-8e41-268bb036a54a/e1dd8a5b-bfac-4fb2-b748-af153c7dae23"
+      (reference "koso-1") (unit 1) (value "Conn_01x03") (footprint "Connector_PinHeader_2.54mm:PinHeader_1x03_P2.54mm_Vertical")
+    )
     (path "/0b22d592-b723-42a2-89dd-bec665c2bd26/4e7e5f68-8854-475b-a33a-14d3a062a224"

Commit message: Fixes and optimizations (unuseful I/O lines dropped)
Connections:
- net i_brakeSwitch: no longer names the net of U4.22 (PC0)
- net o_stopLight: no longer names the net of U4.27 (PC5)
- no-connect marks 6 -> 8
Changed lines of the file:
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@@
   (no_connect (at 142.6464 109.982))
   (no_connect (at 112.1664 64.262))
+  (no_connect (at 142.6464 99.822))
   (no_connect (at 142.6464 66.802))
+  (no_connect (at 142.6464 112.522))
   (no_connect (at 142.6464 64.262))
   (wire (pts (xy 173.482 146.4564) (xy 151.638 146.4564))
@@
     (stroke (width 0) (type default) (color 0 0 0 0))
   )
-  (wire (pts (xy 147.828 98.2472) (xy 147.828 99.822))
-    (stroke (width 0) (type default) (color 0 0 0 0))
-  )
   (wire (pts (xy 147.9296 81.026) (xy 185.4708 81.026))
     (stroke (width 0) (type default) (color 0 0 0 0))
@@
     (stroke (width 0) (type default) (color 0 0 0 0))
   )
-  (wire (pts (xy 142.6464 112.522) (xy 147.1676 112.522))
-    (stroke (width 0) (type default) (color 0 0 0 0))
-  )
   (wire (pts (xy 142.6464 76.962) (xy 190.5 76.962))
     (stroke (width 0) (type default) (color 0 0 0 0))
@@
     (stroke (width 0) (type default) (color 0 0 0 0))
   )
-  (wire (pts (xy 147.1676 112.522) (xy 147.1676 115.062))
-    (stroke (width 0) (type default) (color 0 0 0 0))
-  )
-  (wire (pts (xy 147.828 98.2472) (xy 157.9372 98.2472))
-    (stroke (width 0) (type default) (color 0 0 0 0))
-  )
   (wire (pts (xy 145.1864 151.3332) (xy 180.0352 151.3332))
     (stroke (width 0) (type default) (color 0 0 0 0))
@@
     (stroke (width 0) (type default) (color 0 0 0 0))
   )
-  (wire (pts (xy 147.1676 115.062) (xy 157.9372 115.062))
-    (stroke (width 0) (type default) (color 0 0 0 0))
-  )
   (wire (pts (xy 180.086 136.7028) (xy 173.482 136.7028))
     (stroke (width 0) (type default) (color 0 0 0 0))
@@
   )
   (wire (pts (xy 103.2764 176.53) (xy 108.3564 176.53))
-    (stroke (width 0) (type default) (color 0 0 0 0))
-  )
-  (wire (pts (xy 142.6464 99.822) (xy 147.828 99.822))
     (stroke (width 0) (type default) (color 0 0 0 0))
   )
@@
     )
   )
-  (global_label "o_stopLight" (shape input) (at 157.9372 115.062 0) (fields_autoplaced)
-    (effects (font (size 1.27 1.27)) (justify left))
-    (property "Riferimenti inter-foglio" "${INTERSHEET_REFS}" (id 0) (at 171.1755 114.9826 0)
-      (effects (font (size 1.27 1.27)) (justify left) hide)
-    )
-  )
   (global_label "o_neutral" (shape input) (at 190.6524 100.1268 0) (fields_autoplaced)
     (effects (font (size 1.27 1.27)) (justify left))
@@
     (effects (font (size 1.27 1.27)) (justify left))
     (property "Riferimenti inter-foglio" "${INTERSHEET_REFS}" (id 0) (at 204.3455 86.7886 0)
-      (effects (font (size 1.27 1.27)) (justify left) hide)
-    )
-  )
-  (global_label "i_brakeSwitch" (shape input) (at 157.9372 98.2472 0) (fields_autoplaced)
-    (effects (font (size 1.27 1.27)) (justify left))
-    (property "Riferimenti inter-foglio" "${INTERSHEET_REFS}" (id 0) (at 173.2317 98.1678 0)
       (effects (font (size 1.27 1.27)) (justify left) hide)
     )
@@
       (reference "RA47") (unit 1) (value "3K") (footprint "Resistor_THT:R_Axial_DIN0207_L6.3mm_D2.5mm_P7.62mm_Horizontal")
     )
+    (path "/44e17612-9f2f-476d-8e41-268bb036a54a/9b01f903-96a2-4bcf-9503-26d27170380d"
+      (reference "RA48") (unit 1) (value "100K") (footprint "Resistor_THT:R_Axial_DIN0207_L6.3mm_D2.5mm_P7.62mm_Horizontal")
+    )
+    (path "/44e17612-9f2f-476d-8e41-268bb036a54a/3c45448e-6986-47cd-934b-5c3e13a3dabd"
+      (reference "RA49") (unit 1) (value "100K") (footprint "Resistor_THT:R_Axial_DIN0207_L6.3mm_D2.5mm_P7.62mm_Horizontal")
+    )
     (path "/dfeffa1f-9119-4780-8aed-ab76c9242c17"
       (reference "RV1") (unit 1) (value "10K") (footprint "Potentiometer_THT:Potentiometer_Bourns_3296W_Vertical")
@@
       (reference "RV2") (unit 1) (value "10K") (footprint "Potentiometer_THT:Potentiometer_Bourns_3296W_Vertical")
     )
-    (path "/937463ea-d3fe-417a-91f3-c7891b585b2f/fadd7508-0894-4e7a-a9c8-6bb88b23641e"
-      (reference "RearDevs1") (unit 1) (value "Conn_01x09") (footprint "Connector_PinHeader_2.54mm:PinHeader_1x09_P2.54mm_Vertical")
+    (path "/937463ea-d3fe-417a-91f3-c7891b585b2f/5510d55d-0f19-462b-b63a-fa24c3d3dcc7"
+      (reference "RearDevs1") (unit 1) (value "Conn_01x08") (footprint "Connector_PinHeader_2.54mm:PinHeader_1x08_P2.54mm_Vertical")
     )
     (path "/5aeeaf4d-5399-4718-881e-79b5afe08a8c"

Commit message: fixes...
Parts:
- added C2: 100nF, Capacitor_THT:C_Disc_D4.3mm_W1.9mm_P5.00mm, symbol Device:C
Connections:
- net +5V: now also U4.32 (AREF), C2.1
- net GND: now also C2.2
- net tempPower: no longer U4.30 (AVCC)
Changed lines of the file:
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@@
   (junction (at 80.391 188.087) (diameter 0) (color 0 0 0 0)
   )
+  (junction (at 105.156 69.342) (diameter 0) (color 0 0 0 0)
+  )
   (junction (at 37.211 185.42) (diameter 0) (color 0 0 0 0)
   )
-  (junction (at 127.4064 44.704) (diameter 0) (color 0 0 0 0)
-  )
   (junction (at 108.3564 176.53) (diameter 0) (color 0 0 0 0)
   )
@@
   )
   (no_connect (at 112.1664 59.182))
-  (no_connect (at 112.1664 69.342))
   (no_connect (at 142.6464 109.982))
   (no_connect (at 112.1664 64.262))
@@
   (no_connect (at 142.6464 66.802))
   (no_connect (at 142.6464 112.522))
+  (no_connect (at 129.9464 46.482))
   (no_connect (at 142.6464 64.262))
   (wire (pts (xy 173.482 146.4564) (xy 151.638 146.4564))
@@
     (stroke (width 0) (type default) (color 0 0 0 0))
   )
-  (wire (pts (xy 127.4064 39.37) (xy 127.4064 44.704))
+  (wire (pts (xy 127.4064 39.37) (xy 127.4064 46.482))
     (stroke (width 0) (type default) (color 0 0 0 0))
   )
@@
     (stroke (width 0) (type default) (color 0 0 0 0))
   )
-  (wire (pts (xy 127.4064 44.704) (xy 127.4064 46.482))
-    (stroke (width 0) (type default) (color 0 0 0 0))
-  )
   (wire (pts (xy 149.1488 102.362) (xy 149.1488 101.5492))
     (stroke (width 0) (type default) (color 0 0 0 0))
@@
     (stroke (width 0) (type default) (color 0 0 0 0))
   )
+  (wire (pts (xy 94.742 69.342) (xy 105.156 69.342))
+    (stroke (width 0) (type default) (color 0 0 0 0))
+  )
   (wire (pts (xy 150.5204 92.202) (xy 142.6464 92.202))
     (stroke (width 0) (type default) (color 0 0 0 0))
@@
     (stroke (width 0) (type default) (color 0 0 0 0))
   )
+  (wire (pts (xy 105.156 69.342) (xy 105.156 70.866))
+    (stroke (width 0) (type default) (color 0 0 0 0))
+  )
   (wire (pts (xy 84.836 169.672) (xy 84.836 176.53))
     (stroke (width 0) (type default) (color 0 0 0 0))
@@
     (stroke (width 0) (type default) (color 0 0 0 0))
   )
-  (wire (pts (xy 129.9464 44.704) (xy 127.4064 44.704))
-    (stroke (width 0) (type default) (color 0 0 0 0))
-  )
   (wire (pts (xy 142.6464 125.222) (xy 154.5844 125.222))
     (stroke (width 0) (type default) (color 0 0 0 0))
@@
     (stroke (width 0) (type default) (color 0 0 0 0))
   )
+  (wire (pts (xy 105.156 78.486) (xy 105.156 79.9084))
+    (stroke (width 0) (type default) (color 0 0 0 0))
+  )
   (wire (pts (xy 142.6464 71.882) (xy 161.3916 71.882))
     (stroke (width 0) (type default) (color 0 0 0 0))
@@
     (stroke (width 0) (type default) (color 0 0 0 0))
   )
-  (wire (pts (xy 129.9464 46.482) (xy 129.9464 44.704))
-    (stroke (width 0) (type default) (color 0 0 0 0))
-  )
   (wire (pts (xy 144.6784 117.602) (xy 142.6464 117.602))
     (stroke (width 0) (type default) (color 0 0 0 0))
@@
   )
   (wire (pts (xy 30.988 176.403) (xy 30.988 169.672))
+    (stroke (width 0) (type default) (color 0 0 0 0))
+  )
+  (wire (pts (xy 112.1664 69.342) (xy 105.156 69.342))
     (stroke (width 0) (type default) (color 0 0 0 0))
   )
@@
     )
   )
+  (global_label "+5V" (shape input) (at 94.742 69.342 180) (fields_autoplaced)
+    (effects (font (size 1.27 1.27)) (justify right))
+    (property "Riferimenti inter-foglio" "${INTERSHEET_REFS}" (id 0) (at 88.4584 69.4214 0)
+      (effects (font (size 1.27 1.27)) (justify right) hide)
+    )
+  )
   (global_label "i_horn" (shape input) (at 190.754 90.17 0) (fields_autoplaced)
     (effects (font (size 1.27 1.27)) (justify left))
@@
     )
     (property "Datasheet" "~" (id 3) (at 108.3564 180.8988 0)
+      (effects (font (size 1.27 1.27)) hide)
+    )
+    (pin "1")
+    (pin "2")
+  )
+  (symbol (lib_id "Device:C") (at 105.156 74.676 0) (unit 1)
+    (in_bom yes) (on_board yes)
+    (property "Reference" "C2" (id 0) (at 109.0168 73.4059 0)
+      (effects (font (size 1.27 1.27)) (justify left) hide)
+    )
+    (property "Value" "100nF" (id 1) (at 105.664 77.4192 0)
+      (effects (font (size 1.27 1.27)) (justify left))
+    )
+    (property "Footprint" "Capacitor_THT:C_Disc_D4.3mm_W1.9mm_P5.00mm" (id 2) (at 106.1212 78.486 0)
+      (effects (font (size 1.27 1.27)) hide)
+    )
+    (property "Datasheet" "~" (id 3) (at 105.156 74.676 0)
       (effects (font (size 1.27 1.27)) hide)
     )
@@
     (pin "2")
   )
+  (symbol (lib_id "power:GND") (at 105.156 79.9084 0) (unit 1)
+    (in_bom yes) (on_board yes) (fields_autoplaced)
+    (property "Reference" "#PWR0111" (id 0) (at 105.156 86.2584 0)
+      (effects (font (size 1.27 1.27)) hide)
+    )
+    (property "Value" "GND" (id 1) (at 105.156 85.09 0))
+    (property "Footprint" "" (id 2) (at 105.156 79.9084 0)
+      (effects (font (size 1.27 1.27)) hide)
+    )
+    (property "Datasheet" "" (id 3) (at 105.156 79.9084 0)
+      (effects (font (size 1.27 1.27)) hide)
+    )
+    (pin "1")
+  )
   (symbol (lib_id "power:GND") (at 30.988 185.42 0) (unit 1)
     (in_bom yes) (on_board yes)
@@
       (reference "#PWR0110") (unit 1) (value "+12V") (footprint "")
     )
+    (path "/ceecd370-84cb-4307-84e5-75017587eab5"
+      (reference "#PWR0111") (unit 1) (value "GND") (footprint "")
+    )
     (path "/44e17612-9f2f-476d-8e41-268bb036a54a/ca96e50f-3e2b-4429-a303-34aeefffd5a5"
       (reference "Arrow_p1") (unit 1) (value "Conn_01x03") (footprint "Connector_Wire:SolderWire-1.5sqmm_1x03_P6mm_D1.7mm_OD3mm")
@@
       (reference "C1") (unit 1) (value "C_Polarized_Small") (footprint "Capacitor_THT:CP_Radial_D8.0mm_P2.50mm")
     )
+    (path "/30686728-a02e-4504-8ee7-08ed90242c91"
+      (reference "C2") (unit 1) (value "100nF") (footprint "Capacitor_THT:C_Disc_D4.3mm_W1.9mm_P5.00mm")
+    )
     (path "/30dc0a46-b131-4274-a1fd-5018492748b9"
       (reference "C9") (unit 1) (value "C_Polarized_Small") (footprint "Capacitor_THT:CP_Radial_D8.0mm_P2.50mm")
@@
     )
     (path "/0b22d592-b723-42a2-89dd-bec665c2bd26/b8448d20-86fe-4c18-8be5-bf46157011d9"
-      (reference "R1") (unit 1) (value "500") (footprint "Resistor_THT:R_Axial_DIN0309_L9.0mm_D3.2mm_P12.70mm_Horizontal")
+      (reference "R1") (unit 1) (value "1K") (footprint "Resistor_THT:R_Axial_DIN0207_L6.3mm_D2.5mm_P10.16mm_Horizontal")
     )
     (path "/44e17612-9f2f-476d-8e41-268bb036a54a/066c1919-c2ec-41fd-8aa7-336272f3d1ae"
