File: PCB/pcb-b.kicad_sch (KiCad schematic)
At the start: 11 parts, among them U1 L7805, U2 L7805, U3 L7805

Commit message: fixes
Connections:
- net c_rightArrow: now also to_pcA2.3 (Pin_3)
- net c_engineOFF: now reaches to_pcA2.4 (Pin_4)
- net o_engineON: now reaches to_pcA2.5 (Pin_5)
- no-connect marks 4 -> 5
Other:
- added sheet start-stop (mbes_start_stop.kicad_sch)

Commit message: fixes
Parts:
- to_pcA2, to_pcA3: footprint (none) -> Connector_PinSocket_2.54mm:PinSocket_1x05_P2.54mm_Vertical
- to_pcbA1, to_pcbA4: footprint (none) -> Connector_PinSocket_2.54mm:PinSocket_1x06_P2.54mm_Vertical
