File: PCB/conn_to_pcbb.kicad_sch (KiCad schematic)
At the start: 4 parts

Commit message: fixes
Connections:
- net o_engineON: now reaches to_pcbB2.5 (Pin_5)
- no-connect marks 6 -> 5
Changed lines of the file:
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@@
   (no_connect (at 135.5344 92.8116))
   (no_connect (at 115.1128 80.0608))
-  (no_connect (at 115.1128 95.3516))
   (wire (pts (xy 144.3228 80.6196) (xy 144.3228 80.0608))
     (stroke (width 0) (type default) (color 0 0 0 0))
@@
   )
   (wire (pts (xy 135.5344 77.5208) (xy 145.1356 77.5208))
+    (stroke (width 0) (type default) (color 0 0 0 0))
+  )
+  (wire (pts (xy 98.3488 94.742) (xy 104.5972 94.742))
     (stroke (width 0) (type default) (color 0 0 0 0))
   )
@@
   )
   (wire (pts (xy 143.4084 69.9008) (xy 143.4084 69.2404))
+    (stroke (width 0) (type default) (color 0 0 0 0))
+  )
+  (wire (pts (xy 104.5972 95.3516) (xy 115.1128 95.3516))
     (stroke (width 0) (type default) (color 0 0 0 0))
   )
@@
     (stroke (width 0) (type default) (color 0 0 0 0))
   )
+  (wire (pts (xy 104.5972 94.742) (xy 104.5972 95.3516))
+    (stroke (width 0) (type default) (color 0 0 0 0))
+  )
   (wire (pts (xy 98.5012 91.7448) (xy 103.378 91.7448))
     (stroke (width 0) (type default) (color 0 0 0 0))
@@
     )
   )
+  (global_label "o_engineON" (shape input) (at 98.3488 94.742 180) (fields_autoplaced)
+    (effects (font (size 1.27 1.27)) (justify right))
+    (property "Riferimenti inter-foglio" "${INTERSHEET_REFS}" (id 0) (at 84.929 94.6626 0)
+      (effects (font (size 1.27 1.27)) (justify right) hide)
+    )
+  )

Commit message: Unusefull components removing and RS232 connected also to PCB-b
- The low-pass filter on RS232 RXD has been removed because external serial cable idea has been dropped
- The RS232 lines are been connected also to the PCB-b for future (CH5 module) Bluetooth implementation
Connections:
- net c_RS232_RXD: now reaches to_pcbB2.1 (Pin_1)
- net c_RS232_TXT: now reaches to_pcbB2.2 (Pin_2)
- no-connect marks 5 -> 3
Changed lines of the file:
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@@
   (junction (at 141.1732 74.9808) (diameter 0) (color 0 0 0 0)
   )
-  (no_connect (at 115.1128 87.7316))
   (no_connect (at 115.1128 77.5208))
-  (no_connect (at 115.1128 85.1916))
   (no_connect (at 135.5344 92.8116))
   (no_connect (at 115.1128 80.0608))
+  (wire (pts (xy 106.8324 85.5472) (xy 106.8324 87.7316))
+    (stroke (width 0) (type default) (color 0 0 0 0))
+  )
   (wire (pts (xy 144.3228 80.6196) (xy 144.3228 80.0608))
     (stroke (width 0) (type default) (color 0 0 0 0))
@@
     (stroke (width 0) (type default) (color 0 0 0 0))
   )
+  (wire (pts (xy 108.1532 85.1916) (xy 115.1128 85.1916))
+    (stroke (width 0) (type default) (color 0 0 0 0))
+  )
+  (wire (pts (xy 108.1532 82.4484) (xy 108.1532 85.1916))
+    (stroke (width 0) (type default) (color 0 0 0 0))
+  )
   (wire (pts (xy 141.1732 74.93) (xy 141.1732 74.9808))
     (stroke (width 0) (type default) (color 0 0 0 0))
@@
     (stroke (width 0) (type default) (color 0 0 0 0))
   )
+  (wire (pts (xy 98.4504 82.4484) (xy 108.1532 82.4484))
+    (stroke (width 0) (type default) (color 0 0 0 0))
+  )
   (wire (pts (xy 103.1748 74.1172) (xy 103.1748 72.4408))
     (stroke (width 0) (type default) (color 0 0 0 0))
@@
     (stroke (width 0) (type default) (color 0 0 0 0))
   )
+  (wire (pts (xy 106.8324 87.7316) (xy 115.1128 87.7316))
+    (stroke (width 0) (type default) (color 0 0 0 0))
+  )
   (wire (pts (xy 104.9528 77.5208) (xy 104.9528 74.9808))
     (stroke (width 0) (type default) (color 0 0 0 0))
@@
     (stroke (width 0) (type default) (color 0 0 0 0))
   )
+  (wire (pts (xy 98.3996 85.5472) (xy 106.8324 85.5472))
+    (stroke (width 0) (type default) (color 0 0 0 0))
+  )
   (wire (pts (xy 150.9776 95.3516) (xy 150.9776 95.4024))
     (stroke (width 0) (type default) (color 0 0 0 0))
@@
     )
   )
+  (global_label "c_RS232_TXT" (shape input) (at 98.3996 85.5472 180) (fields_autoplaced)
+    (effects (font (size 1.27 1.27)) (justify right))
+    (property "Riferimenti inter-foglio" "${INTERSHEET_REFS}" (id 0) (at 83.7098 85.4678 0)
+      (effects (font (size 1.27 1.27)) (justify right) hide)
+    )
+  )
   (global_label "+5V" (shape input) (at 98.3488 74.1172 180) (fields_autoplaced)
     (effects (font (size 1.27 1.27)) (justify right))
@@
     )
   )
+  (global_label "c_RS232_RXD" (shape input) (at 98.4504 82.4484 180) (fields_autoplaced)
+    (effects (font (size 1.27 1.27)) (justify right))
+    (property "Riferimenti inter-foglio" "${INTERSHEET_REFS}" (id 0) (at 83.1559 82.369 0)
+      (effects (font (size 1.27 1.27)) (justify right) hide)
+    )
+  )
