File: PCB/pcb-c/pcb-c.kicad_pcb (KiCad board)
At the start: 2 copper layers, 45.2 x 34.8 mm, 37 parts, among them Q1 BC817, Q13 TPCA8120,L1Q, Q2 TPCA8120,L1Q, Q3 BC817, Q4 BC817, Q5 TPCA8120,L1Q, Q6 BC817, Q7 TPCA8120,L1Q, Q8 BC817, Q9 TPCA8120,L1Q

Commit message: Floating FET's source pin fixed
The pin was in floating state when the associated fuse is temporary off
Parts:
- added R11: 100K, Resistor_SMD:R_1206_3216Metric, B.Cu at (178.6, 97.3)
- added R15: 100K, Resistor_SMD:R_1206_3216Metric, B.Cu at (173.6, 97.3)
- added R19: 100K, Resistor_SMD:R_1206_3216Metric, B.Cu at (189.8, 100.0)
- added R3: 100K, Resistor_SMD:R_1206_3216Metric, B.Cu at (172.1, 105.1)
- added R6: 100K, Resistor_SMD:R_1206_3216Metric, B.Cu at (159.8, 107.3)
- D1: value D_Small -> M7
- moved R14 1.73 mm to (176.1, 97.3), turned to -90 degrees
Routing:
- net +12V: track 79.5 -> 95.8 mm
- net Net-(Q13-S_1): track 18.6 -> 14.4 mm
- net Net-(Q5-S_1): track 12.4 -> 15.8 mm
- net Net-(Q9-S_1): track 9.09 -> 11.9 mm
- net Net-(Q7-S_1): track 10.7 -> 13.0 mm
