File: PCB/pcb-c/pcb-c.kicad_pcb (KiCad board)
At the start: 2 copper layers, 45.2 x 34.8 mm, 42 parts, among them Q1 BC817, Q13 TPCA8120,L1Q, Q2 TPCA8120,L1Q, Q3 BC817, Q4 BC817, Q5 TPCA8120,L1Q, Q6 BC817, Q7 TPCA8120,L1Q, Q8 BC817, Q9 TPCA8120,L1Q

Commit message: Small optimization
Parts:
- R13, R17, R4, R7, R9: value 10K -> 15K
Changed lines of the file:
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@@
 			)
 		)
-		(property "Value" "10K"
+		(property "Value" "15K"
 			(at 0 0 90)
 			(layer "F.Fab")
@@
 			)
 		)
-		(property "Value" "10K"
+		(property "Value" "15K"
 			(at 0 0 90)
 			(layer "F.Fab")
@@
 			)
 		)
-		(property "Value" "10K"
+		(property "Value" "15K"
 			(at 0 0 90)
 			(layer "F.Fab")
@@
 			)
 		)
-		(property "Value" "10K"
+		(property "Value" "15K"
 			(at 0 0 90)
 			(layer "F.Fab")
@@
 			)
 		)
-		(property "Value" "10K"
+		(property "Value" "15K"
 			(at 0 0 90)
 			(layer "F.Fab")
