File: PCB/pcb-c/pcb-c.kicad_sch (KiCad schematic)
At the start: 42 parts, among them Q1 BC817, Q13 TPCA8120,L1Q, Q2 TPCA8120,L1Q, Q3 BC817, Q4 BC817, Q5 TPCA8120,L1Q, Q6 BC817, Q7 TPCA8120,L1Q, Q8 BC817, Q9 TPCA8120,L1Q

Commit message: Small optimization
Parts:
- R13, R17, R4, R7, R9: value 10K -> 15K
Changed lines of the file:
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@@
 			)
 		)
-		(property "Value" "10K"
+		(property "Value" "15K"
 			(at 154.178 82.804 90)
 			(effects
@@
 			)
 		)
-		(property "Value" "10K"
+		(property "Value" "15K"
 			(at 46.228 39.878 90)
 			(effects
@@
 			)
 		)
-		(property "Value" "10K"
+		(property "Value" "15K"
 			(at 44.958 126.238 90)
 			(effects
@@
 			)
 		)
-		(property "Value" "10K"
+		(property "Value" "15K"
 			(at 151.638 41.148 90)
 			(effects
@@
 			)
 		)
-		(property "Value" "10K"
+		(property "Value" "15K"
 			(at 45.72 82.804 90)
 			(effects
